File: RotatorController.kicad_sch (KiCad schematic)
At the start: 58 parts, among them J1 USB_A, J2 Rotator, J4 Motor Cap, K1 G5LE-1, K2 G5LE-1, K3 G5LE-1, Q1 BSS123, Q2 BSS123, Q3 BSS123, SW1 CW, SW2 CW, U1 Teensy4.0, U3 AP2161W

Commit message: finish cleanup of deleted and renamed datasheets, stage and commits trivial changes to pcb and sch
Parts:
- removed D1, D2: BAS40-04, Package_TO_SOT_SMD:SOT-23, symbol Diode:BAS40-04
- removed D19: 5V, LED_SMD:LED_miniPLCC_2315_Handsoldering, symbol LED:IR204A
- removed J1: USB_A, Connector_USB:USB_A_TE_292303-7_Horizontal, symbol Connector:USB_A
- removed J4: Motor Cap, Connector_PinHeader_2.54mm:PinHeader_1x02_P2.54mm_Vertical, symbol Connector:Conn_01x02_Socket
- removed R15: 560, Resistor_SMD:R_0805_2012Metric_Pad1.20x1.40mm_HandSolder, symbol Device:R_Small_US
- removed U3: AP2161W, Package_TO_SOT_SMD:SOT-23-5, symbol Power_Management:AP2161W
- added J3: Controller, Connector_TE-Connectivity:TE_MATE-N-LOK_1-770970-x_2x04_P4.14mm_Horizontal, symbol Connector:Conn_01x08_Pin
- J2: symbol Connector:Conn_01x10_Socket -> Connector:Conn_01x10_Pin
Connections:
- net Cap1: now also J3.5 (Pin_5)
- net Cap2: now also J3.1 (Pin_1)
- no-connect marks 17 -> 16
Other:
- note added: "Capacitor Option Select"
- note added: "Manual Controller Interface"
- note added: "Meter Driver"
- note added: "Motor Switch Interface"
- note added: "Option for this controller placed inline with manual control box Capacitor in manual box used Meter driven by PWM Detect 26 VAC Provided by switches No need to use brake switch Use 26 VAC supplied by control box"
- note added: "Pins assigned for best PCB layout"
- note added: "Rotator Controller, WA1HCO, Inline option"
- note removed: "Controller interface, 5V and serial"
- moved on the sheet: O1
