File: Rotator-Controller-V4.kicad_sch (KiCad schematic)
At the start: 92 parts, among them J1 Serial, J2 Rotator, J3 USB-C 2.0 16P, J4 Motor Cap, J6 Header 1x3, SW1 CW, SW2 CW, U1 ATtiny1616-M, U2 AP2161W, U3 CPC1966, U4 CPC1966, U5 CPC1966, U6 ADUM3160, U7 FT231XQ, U8 NDP6802SF-50, U9 STM32F301K8Tx

Commit message: More work on schematic Started software conversion to STM32F405 MCU
Parts:
- removed C1: 0.1 200V, Capacitor_SMD:C_1206_3216Metric_Pad1.33x1.80mm_HandSolder, symbol Device:C_Small
- removed C15, C19: .1u, Capacitor_SMD:C_0402_1005Metric, symbol Device:C
- removed D19: 5V, LED_SMD:LED_0402_1005Metric, symbol LED:IR204A
- removed D20, D21: Yellow, LED_SMD:LED_0402_1005Metric, symbol Device:LED
- removed D9: 2BZX84C3V6, Package_TO_SOT_SMD:SOT-23, symbol Diode:MMBZxx
- removed J1: Serial, Connector_USB:USB_A_TE_292303-7_Horizontal, symbol Connector:USB_A
- removed J6: Header 1x3, Connector_PinHeader_2.54mm:PinHeader_1x03_P2.54mm_Vertical, symbol Connector:Conn_01x03_Pin
- removed R15: 560, Resistor_SMD:R_0402_1005Metric, symbol Device:R_Small_US
- removed R26, R27, R28, R29: 1K, Resistor_SMD:R_0402_1005Metric, symbol Device:R_US
- removed U1: ATtiny1616-M, Package_DFN_QFN:VQFN-20-1EP_3x3mm_P0.4mm_EP1.7x1.7mm, symbol MCU_Microchip_ATtiny:ATtiny1616-M
- removed U2: AP2161W, Package_TO_SOT_SMD:SOT-23-5, symbol Power_Management:AP2161W
- removed U7: FT231XQ, Package_DFN_QFN:QFN-20-1EP_4x4mm_P0.5mm_EP2.5x2.5mm, symbol Interface_USB:FT231XQ
- removed U9: STM32F301K8Tx, Package_QFP:LQFP-32_7x7mm_P0.8mm, symbol MCU_ST_STM32F3:STM32F301K8Tx
- added C11, C16, C18, C8: 100n, Capacitor_SMD:C_0603_1608Metric, symbol Device:C_Small
- added C12, C15: 2.2u, Capacitor_SMD:C_0603_1608Metric, symbol Device:C_Small
- added C17, C33: 10u, Capacitor_SMD:C_0603_1608Metric, symbol Device:C_Small
- added C29: 0.1 200V, Capacitor_SMD:C_1206_3216Metric_Pad1.33x1.80mm_HandSolder, symbol Device:C_Small
- added C34: 1u, Capacitor_SMD:C_0603_1608Metric, symbol Device:C_Small
- added C5: 4.7u, Capacitor_SMD:C_0603_1608Metric, symbol Device:C_Small
- added C6: 0.1u, Capacitor_SMD:C_0603_1608Metric, symbol Device:C_Small
- added FB2: FerriteBead_Small, Inductor_SMD:L_0805_2012Metric, symbol Device:FerriteBead_Small
- added R26, R8: 10K, Resistor_SMD:R_0603_1608Metric, symbol Device:R_Small_US
- added R5, R6: 27, Resistor_SMD:R_0402_1005Metric, symbol Device:R_US
- added U2: STM32F405RGTx, Package_QFP:LQFP-64_10x10mm_P0.5mm, symbol MCU_ST_STM32F4:STM32F405RGTx
- added U7: AP2112K-3.3, Package_TO_SOT_SMD:SOT-23-5, symbol Regulator_Linear:AP2112K-3.3
- added Y1: 12M, Crystal:Crystal_SMD_2016-4Pin_2.0x1.6mm, symbol Device:Crystal_GND24_Small
- C1: renamed from C16; footprint Capacitor_SMD:C_0402_1005Metric -> Capacitor_SMD:C_0603_1608Metric
- C10, C13: value 0.1 -> 20p; footprint Capacitor_SMD:C_1206_3216Metric_Pad1.33x1.80mm_HandSolder -> Capacitor_SMD:C_0603_1608Metric
- C14: value 120u -> 100n; footprint Capacitor_SMD:C_1206_3216Metric_Pad1.33x1.80mm_HandSolder -> Capacitor_SMD:C_0603_1608Metric
- C2: renamed from C20; footprint Capacitor_SMD:C_0402_1005Metric -> Capacitor_SMD:C_0603_1608Metric
- C3: renamed from C18; footprint Capacitor_SMD:C_0402_1005Metric -> Capacitor_SMD:C_0603_1608Metric
- C4: renamed from C25; footprint Capacitor_SMD:C_0402_1005Metric -> Capacitor_SMD:C_0603_1608Metric
- C7: renamed from C24; footprint Capacitor_SMD:C_0402_1005Metric -> Capacitor_SMD:C_0603_1608Metric
- C9: renamed from C17; footprint Capacitor_SMD:C_0402_1005Metric -> Capacitor_SMD:C_0603_1608Metric
- D4: renamed from D10; value White -> 5V_GRN
- R1: renamed from R10; footprint Resistor_SMD:R_0402_1005Metric -> Resistor_SMD:R_0603_1608Metric
- R10: renamed from R5; footprint Resistor_SMD:R_0402_1005Metric -> Resistor_SMD:R_0603_1608Metric
- R11: renamed from R20; value 1K5 -> 1K; footprint Resistor_SMD:R_0402_1005Metric -> Resistor_SMD:R_0603_1608Metric
- R12: renamed from R3; value 1k5 -> 1k; footprint Resistor_SMD:R_0402_1005Metric -> Resistor_SMD:R_0603_1608Metric
- R13: renamed from R19; value 1K5 -> 1K; footprint Resistor_SMD:R_0402_1005Metric -> Resistor_SMD:R_0603_1608Metric
- R14: renamed from R16; value 1K5 -> 1K; footprint Resistor_SMD:R_0402_1005Metric -> Resistor_SMD:R_0603_1608Metric
- R15: renamed from R18; value 1K5 -> 1K; footprint Resistor_SMD:R_0402_1005Metric -> Resistor_SMD:R_0603_1608Metric
- R16: renamed from R17; value 1K5 -> 1K; footprint Resistor_SMD:R_0402_1005Metric -> Resistor_SMD:R_0603_1608Metric
- R17: renamed from R1; footprint Resistor_SMD:R_0402_1005Metric -> Resistor_SMD:R_0603_1608Metric
- R18: renamed from R6; footprint Resistor_SMD:R_0402_1005Metric -> Resistor_SMD:R_0603_1608Metric
- R19: renamed from R8; footprint Resistor_SMD:R_0402_1005Metric -> Resistor_SMD:R_0603_1608Metric
- R2: renamed from R21; footprint Resistor_SMD:R_0402_1005Metric -> Resistor_SMD:R_0603_1608Metric
- R20: renamed from R7; footprint Resistor_SMD:R_0402_1005Metric -> Resistor_SMD:R_0603_1608Metric
- R21: renamed from R9; footprint Resistor_SMD:R_0402_1005Metric -> Resistor_SMD:R_0603_1608Metric
- R22: renamed from R11; footprint Resistor_SMD:R_0402_1005Metric -> Resistor_SMD:R_0603_1608Metric
- R23: renamed from R12; footprint Resistor_SMD:R_0402_1005Metric -> Resistor_SMD:R_0603_1608Metric
- R24: renamed from R13; footprint Resistor_SMD:R_0402_1005Metric -> Resistor_SMD:R_0603_1608Metric
- R25: renamed from R14; footprint Resistor_SMD:R_0402_1005Metric -> Resistor_SMD:R_0603_1608Metric
- R3: renamed from R22; footprint Resistor_SMD:R_0402_1005Metric -> Resistor_SMD:R_0603_1608Metric
- R4: renamed from R2; footprint Resistor_SMD:R_0402_1005Metric -> Resistor_SMD:R_0603_1608Metric
- R7: renamed from R25; footprint Resistor_SMD:R_0402_1005Metric -> Resistor_SMD:R_0603_1608Metric
- R9: renamed from R4; footprint Resistor_SMD:R_0402_1005Metric -> Resistor_SMD:R_0603_1608Metric
- renumbered C21 to C19, C2 to C20, C3 to C21, C4 to C22, C5 to C23, C6 to C24, C7 to C25, C23 to C26, C8 to C27, C9 to C28, C22 to C30, C11 to C31, C12 to C32, D8 to D1, D13 to D10, D5 to D11, D3 to D12, D18 to D13, D17 to D14, D16 to D15, D14 to D16, D15 to D17, D11 to D2, D7 to D3, D12 to D5, D1 to D6, D4 to D7, D6 to D8, D2 to D9, J3 to J1, J4 to J2, J2 to J3, U6 to U1, U8 to U6
Connections:
- net Return is gone; now on net GND: D12.1 (A1), J3.10 (Pin_10), J3.6 (Pin_6)
- net 26VAC: now also C29.1
- net 3V3: no longer R24.1, R25.1
- net 5V: now also R26.1, U7.1 (VIN); no longer C10.1, C9.1, U1.16 (VBUS2)
- net GND: now also C11.2, C12.2, C15.2, C16.2, C17.2, C18.2, C29.2, C33.2, C34.2, C5.2, C6.2, C8.2, R8.1, U2.12 (VSSA), U2.18 (VSS), U2.28 (PB2), U2.63 (VSS), U7.2 (GND), Y1.2, Y1.4
- net at C1.1, D2.1 (K), J1.A7 (D-)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: now also R5.2; no longer U1.7 (UD+)
- net at C3.1, D1.1 (K), J1.A6 (D+)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: now also R6.2; no longer U1.6 (UD-)
- net +3v3: now reaches C7.1, U1.12 (PIN), U1.14 (VDD2)
- net +3v3: now also C9.1, U1.16 (VBUS2), C33.1, C34.1, U7.5 (VOUT)
- net 5VD renamed VBUS
- net 5V_Serial: no longer names the net of C13.1
- net 5V_Serial: now also U2.6 (PH1), Y1.3; no longer C14.1
- net D+M renamed D+
- net D+: now also U2.45 (PA12)
- net D-M renamed D-
- net D-: now also U2.44 (PA11)
- new net: R6.1, U1.7 (UD+)
- new net: C15.1, U2.47 (VCAP_2)
- new net: C12.1, U2.31 (VCAP_1)
- new net: C10.1, U2.5 (PH0), Y1.1
- new net: R8.2, U2.60 (BOOT0)
- new net: C6.1, U2.7 (NRST)
- new net: R26.2, U7.3 (EN)
- new net: R5.1, U1.6 (UD-)
- new net +3V3: C11.1, C14.1, C16.1, C5.1, C8.1, FB2.1, R24.1, R25.1, U2.19 (VDD), U2.32 (VDD), U2.48 (VDD), U2.64 (VDD)
- new net AVCC: C17.1, C18.1, FB2.2, U2.13 (VDDA)
- no-connect marks 12 -> 4
Other:
- note removed: "CBUS signals use defaults"
- note removed: "Comms"
- note removed: "Controller interface, 5V and serial"
- note removed: "Current MCU LEDs USB isolator 8 ma"
- note removed: "Program"
- moved on the sheet: C1, C19, C2, C20, C21, C22, C23, C24, C25, C26, C27, C28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
